File: archivos_kicad/amplificador_V2/amplificacion.kicad_sch (KiCad schematic)
At the start: 24 parts, among them J1 INPUT_L, J2 OUTPUT_L, J3 ALIMENTACION REJILLA, J4 ALIMENTACION FILAMENTO, J5 INPUT_R, J6 OUTPUT_R

Commit message: Add files via upload
Parts:
- RV1, RV2: footprint Potentiometer_THT:Potentiometer_Piher_PC-16_Single_Horizontal -> lib_rama:TRIM_WH148-1A-2-18T-L20
Changed lines of the file:
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@@
 			)
 		)
-		(property "Footprint" "Potentiometer_THT:Potentiometer_Piher_PC-16_Single_Horizontal"
+		(property "Footprint" "lib_rama:TRIM_WH148-1A-2-18T-L20"
 			(at 214.63 88.9 0)
 			(effects
@@
 			)
 		)
-		(property "Footprint" "Potentiometer_THT:Potentiometer_Piher_PC-16_Single_Horizontal"
+		(property "Footprint" "lib_rama:TRIM_WH148-1A-2-18T-L20"
 			(at 200.66 212.09 0)
 			(effects
